Commit message: nav2 and imu added

File: description/lidar.xacro (robot description, xacro)
@@ -4,5 +4,5 @@
         <parent link="chassis"/>
         <child link="laser_frame"/>
-        <origin xyz="0.122 0 0.212" rpy="0 0 0"/>
+        <origin xyz="0.57 0 0.18" rpy="0 0 0"/>
     </joint>
     <link name="laser_frame">

File: description/robot.urdf.xacro (robot description, xacro)
@@ -11,3 +11,4 @@
     </xacro:unless>
     <xacro:include filename="lidar.xacro" />
+    <xacro:include filename="imu.xacro" />
 </robot>

File: description/robot_core.xacro (robot description, xacro)
@@ -2,20 +2,18 @@
 <robot xmlns:xacro="http://www.ros.org/wiki/xacro" >
     <xacro:include filename="inertial_macros.xacro"/>
-    <!--
- <xacro:property name="chassis_length" value="0.6"/>
+    <xacro:property name="chassis_length" value="0.6"/>
     <xacro:property name="chassis_width" value="0.6"/>
     <xacro:property name="chassis_height" value="0.15"/>
     <xacro:property name="chassis_mass" value="0.5"/>
     <xacro:property name="wheel_radius" value="0.0625"/>
-    <xacro:property name="wheel_thickness" value="0.051"/>
+    <xacro:property name="wheel_thickness" value="0.03"/>
     <xacro:property name="wheel_mass" value="1.0"/>
     <xacro:property name="wheel_offset_x" value="0.3"/>
-    <xacro:property name="wheel_offset_y" value="0.3255"/>
-    <xacro:property name="wheel_offset_z" value="-0.06"/>
+    <xacro:property name="wheel_offset_y" value="0.326"/>
+    <xacro:property name="wheel_offset_z" value="-0.0625"/>
     <xacro:property name="caster_wheel_radius" value="0.05"/>
     <xacro:property name="caster_wheel_mass" value="0.5"/>
-    <xacro:property name="caster_wheel_offset_x" value="0.55"/>
+    <xacro:property name="caster_wheel_offset_x" value="0.555"/>
     <xacro:property name="caster_wheel_offset_z" value="${wheel_offset_z - wheel_radius + caster_wheel_radius}"/>
-    -->
     <!-- <xacro:property name="chassis_length" value="0.3"/>
     <xacro:property name="chassis_width" value="0.3"/>
@@ -32,5 +30,5 @@
     <xacro:property name="caster_wheel_offset_x" value="0.24"/>
     <xacro:property name="caster_wheel_offset_z" value="${wheel_offset_z - wheel_radius + caster_wheel_radius}"/> -->
-    <xacro:property name="chassis_length" value="0.335"/>
+    <!-- <xacro:property name="chassis_length" value="0.335"/>
     <xacro:property name="chassis_width" value="0.265"/>
     <xacro:property name="chassis_height" value="0.138"/>
@@ -45,5 +43,5 @@
     <xacro:property name="caster_wheel_mass" value="0.01"/>
     <xacro:property name="caster_wheel_offset_x" value="0.075"/>
-    <xacro:property name="caster_wheel_offset_z" value="${wheel_offset_z - wheel_radius + caster_wheel_radius}"/>
+    <xacro:property name="caster_wheel_offset_z" value="${wheel_offset_z - wheel_radius + caster_wheel_radius}"/> -->
     <material name="white">
         <color rgba="1 1 1 1"/>
@@ -94,5 +92,5 @@
     </link>
     <gazebo reference ="chassis">
-        <material>Gazebo/Orange</material>
+        <material>Gazebo/OrangeTransparent</material>
     </gazebo>
     <!-- LEFT WHEEL LINK-->
